File: Micro_level_PCB_2.0.kicad_sch (KiCad schematic)
At the start: 105 parts, among them J5 Conn_01x06, J6 Conn_01x07_Female, Q1 SI2304DDS, Q2 SI2304DDS, Q3 SI2304DDS, Q4 SI2304DDS, Q5 SI2304DDS, SW1 FSM2JSMAA, SW2 FSM2JSMAA, SW3 FSM2JSMAA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

Commit message: 4 button up/down
Parts:
- added SW6, SW7: FSM2JSMAA, MY_KICAD_LIB:SW_Push_1P1T_NO_6x6mm_H5.0mm, symbol MY_KICAD_SCH:FSM2JSMAA
- D1: value SMF18A -> 1PGSMA4740HR3G
- renumbered Dim to Dim1, Power to Power1, Sensors to Sensors1, Solenoids to Solenoids1
Connections:
- net REMOTE_CAMP is gone; now on net REMOTE_RU: U1.43 (PB3)
- net GND: now also SW6.3 (B), SW6.4 (B), SW7.3 (B), SW7.4 (B)
- net REMOTE_RU: no longer U1.44 (PB4)
- net DOWN renamed Right_DOWN
- net OUTSIDE_VALID: no longer names the net of J6.7 (Pin_7)
- net POWERUP: no longer names the net of U1.11 (PD2)
- net REMOTE_DOWN: no longer names the net of U1.2 (PB6)
- net REMOTE_TRAVEL renamed Left_UP
- net Left_UP: now also SW7.1 (A), SW7.2 (A)
- net REMOTE_UP: no longer names the net of U1.3 (PB7)
- net SPARE1: no longer names the net of U1.25 (PC6)
- net UP renamed Right_UP
- new net Left_DOWN: SW6.1 (A), SW6.2 (A), U1.44 (PB4)
- no-connect marks 19 -> 16

Commit message: move buttons, change jtag connector
Parts:
- removed CX1: Conn2x5_CNC#3220-10-0100-00, Connector_PinSocket_1.27mm:PinSocket_2x05_P1.27mm_Vertical, symbol MY_KICAD_SCH:Conn2x5_CNC#3220-10-0100-00
- added J1: Conn_01x07_Female, Connector_PinHeader_2.54mm:PinHeader_1x07_P2.54mm_Vertical, symbol Connector:Conn_01x07_Female
- renumbered Solenoids1 to J2, Dim1 to J3, Power1 to J4, Sensors1 to j7
Connections:
- net GND: now also J1.7 (Pin_7)
- net RESET: now also J1.6 (Pin_6)
- net TCK: now also J1.1 (Pin_1)
- net TDI: now also J1.4 (Pin_4)
- net TDO: now also J1.3 (Pin_3)
- net TMS: now also J1.2 (Pin_2)
- net V5: now also J1.5 (Pin_5)
- no-connect marks 16 -> 14

Commit message: 4 up/down buttons, remove 2x5 jtag
Connections:
- net CALIBRATE renamed BTN_CALIBRATE
- net CAMP renamed BTN_CAMP
- net Left_DOWN renamed BTN_Left_DOWN
- net Left_UP renamed BTN_Left_UP
- net Right_DOWN renamed BTN_Right_DOWN
- net Right_UP renamed BTN_Right_UP
- net TRAVEL renamed BTN_TRAVEL
Changed lines of the file:
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@@
     )
   )
-  (global_label "CALIBRATE" (shape input) (at 276.86 82.55 180) (fields_autoplaced)
-    (effects (font (size 1.27 1.27)) (justify right))
-    (property "Intersheet References" "${INTERSHEET_REFS}" (id 0) (at 264.7102 82.4706 0)
+  (global_label "BTN_CALIBRATE" (shape input) (at 276.86 82.55 180) (fields_autoplaced)
+    (effects (font (size 1.27 1.27)) (justify right))
+    (property "Intersheet References" "${INTERSHEET_REFS}" (id 0) (at 260.1745 82.4706 0)
       (effects (font (size 1.27 1.27)) (justify right) hide)
     )
@@
     )
   )
-  (global_label "Right_UP" (shape input) (at 277.495 120.015 180) (fields_autoplaced)
-    (effects (font (size 1.27 1.27)) (justify right))
-    (property "Intersheet References" "${INTERSHEET_REFS}" (id 0) (at 266.6152 119.9356 0)
+  (global_label "BTN_Right_UP" (shape input) (at 277.495 120.015 180) (fields_autoplaced)
+    (effects (font (size 1.27 1.27)) (justify right))
+    (property "Intersheet References" "${INTERSHEET_REFS}" (id 0) (at 262.0795 119.9356 0)
       (effects (font (size 1.27 1.27)) (justify right) hide)
     )
@@
     )
   )
-  (global_label "COMP" (shape input) (at 201.93 121.92 0) (fields_autoplaced)
+  (global_label "COMP" (shape output) (at 201.93 121.92 0) (fields_autoplaced)
     (effects (font (size 1.27 1.27)) (justify left))
     (property "Intersheet References" "${INTERSHEET_REFS}" (id 0) (at 209.665 121.8406 0)
@@
     )
   )
-  (global_label "CALIBRATE" (shape input) (at 203.2 137.16 0) (fields_autoplaced)
-    (effects (font (size 1.27 1.27)) (justify left))
-    (property "Intersheet References" "${INTERSHEET_REFS}" (id 0) (at 215.3498 137.0806 0)
+  (global_label "BTN_CALIBRATE" (shape input) (at 203.2 137.16 0) (fields_autoplaced)
+    (effects (font (size 1.27 1.27)) (justify left))
+    (property "Intersheet References" "${INTERSHEET_REFS}" (id 0) (at 219.8855 137.0806 0)
       (effects (font (size 1.27 1.27)) (justify left) hide)
     )
@@
     )
   )
-  (global_label "Left_UP" (shape input) (at 277.5966 138.9888 180) (fields_autoplaced)
-    (effects (font (size 1.27 1.27)) (justify right))
-    (property "Intersheet References" "${INTERSHEET_REFS}" (id 0) (at 268.0473 138.9094 0)
-      (effects (font (size 1.27 1.27)) (justify right) hide)
-    )
-  )
-  (global_label "CAMP" (shape input) (at 203.2 139.7 0) (fields_autoplaced)
-    (effects (font (size 1.27 1.27)) (justify left))
-    (property "Intersheet References" "${INTERSHEET_REFS}" (id 0) (at 210.6931 139.6206 0)
+  (global_label "BTN_Left_UP" (shape input) (at 277.5966 138.9888 180) (fields_autoplaced)
+    (effects (font (size 1.27 1.27)) (justify right))
+    (property "Intersheet References" "${INTERSHEET_REFS}" (id 0) (at 263.5116 138.9094 0)
+      (effects (font (size 1.27 1.27)) (justify right) hide)
+    )
+  )
+  (global_label "BTN_CAMP" (shape input) (at 203.2 139.7 0) (fields_autoplaced)
+    (effects (font (size 1.27 1.27)) (justify left))
+    (property "Intersheet References" "${INTERSHEET_REFS}" (id 0) (at 215.2288 139.6206 0)
       (effects (font (size 1.27 1.27)) (justify left) hide)
     )
@@
     )
   )
-  (global_label "LD" (shape input) (at 201.93 73.66 0) (fields_autoplaced)
+  (global_label "LD" (shape output) (at 201.93 73.66 0) (fields_autoplaced)
     (effects (font (size 1.27 1.27)) (justify left))
     (property "Intersheet References" "${INTERSHEET_REFS}" (id 0) (at 206.6412 73.5806 0)
@@
     )
   )
-  (global_label "RU" (shape input) (at 201.93 71.12 0) (fields_autoplaced)
+  (global_label "RU" (shape output) (at 201.93 71.12 0) (fields_autoplaced)
     (effects (font (size 1.27 1.27)) (justify left))
     (property "Intersheet References" "${INTERSHEET_REFS}" (id 0) (at 206.9436 71.0406 0)
@@
     )
   )
-  (global_label "Right_DOWN" (shape input) (at 203.2 142.24 0) (fields_autoplaced)
-    (effects (font (size 1.27 1.27)) (justify left))
-    (property "Intersheet References" "${INTERSHEET_REFS}" (id 0) (at 216.8617 142.1606 0)
+  (global_label "BTN_Right_DOWN" (shape input) (at 203.2 142.24 0) (fields_autoplaced)
+    (effects (font (size 1.27 1.27)) (justify left))
+    (property "Intersheet References" "${INTERSHEET_REFS}" (id 0) (at 221.3974 142.1606 0)
       (effects (font (size 1.27 1.27)) (justify left) hide)
     )
@@
     )
   )
-  (global_label "Left_UP" (shape input) (at 204.216 93.98 0) (fields_autoplaced)
-    (effects (font (size 1.27 1.27)) (justify left))
-    (property "Intersheet References" "${INTERSHEET_REFS}" (id 0) (at 213.7653 93.9006 0)
+  (global_label "BTN_Left_UP" (shape input) (at 204.216 93.98 0) (fields_autoplaced)
+    (effects (font (size 1.27 1.27)) (justify left))
+    (property "Intersheet References" "${INTERSHEET_REFS}" (id 0) (at 218.301 93.9006 0)
       (effects (font (size 1.27 1.27)) (justify left) hide)
     )
@@
     )
   )
-  (global_label "Left_DOWN" (shape input) (at 204.0636 91.4654 0) (fields_autoplaced)
-    (effects (font (size 1.27 1.27)) (justify left))
-    (property "Intersheet References" "${INTERSHEET_REFS}" (id 0) (at 216.3948 91.386 0)
+  (global_label "BTN_Left_DOWN" (shape input) (at 204.0636 91.4654 0) (fields_autoplaced)
+    (effects (font (size 1.27 1.27)) (justify left))
+    (property "Intersheet References" "${INTERSHEET_REFS}" (id 0) (at 220.9305 91.386 0)
       (effects (font (size 1.27 1.27)) (justify left) hide)
     )
@@
     )
   )
-  (global_label "RD" (shape input) (at 201.93 68.58 0) (fields_autoplaced)
+  (global_label "RD" (shape output) (at 201.93 68.58 0) (fields_autoplaced)
     (effects (font (size 1.27 1.27)) (justify left))
     (property "Intersheet References" "${INTERSHEET_REFS}" (id 0) (at 206.8831 68.5006 0)
@@
     )
   )
-  (global_label "Left_DOWN" (shape input) (at 277.5966 130.0988 180) (fields_autoplaced)
-    (effects (font (size 1.27 1.27)) (justify right))
-    (property "Intersheet References" "${INTERSHEET_REFS}" (id 0) (at 265.2654 130.0194 0)
+  (global_label "BTN_Left_DOWN" (shape input) (at 277.5966 130.0988 180) (fields_autoplaced)
+    (effects (font (size 1.27 1.27)) (justify right))
+    (property "Intersheet References" "${INTERSHEET_REFS}" (id 0) (at 260.7297 130.0194 0)
       (effects (font (size 1.27 1.27)) (justify right) hide)
     )
@@
     )
   )
-  (global_label "CAMP" (shape input) (at 276.86 92.075 180) (fields_autoplaced)
-    (effects (font (size 1.27 1.27)) (justify right))
-    (property "Intersheet References" "${INTERSHEET_REFS}" (id 0) (at 269.3669 91.9956 0)
+  (global_label "BTN_CAMP" (shape input) (at 276.86 92.075 180) (fields_autoplaced)
+    (effects (font (size 1.27 1.27)) (justify right))
+    (property "Intersheet References" "${INTERSHEET_REFS}" (id 0) (at 264.8312 91.9956 0)
       (effects (font (size 1.27 1.27)) (justify right) hide)
     )
@@
     )
   )
-  (global_label "Right_UP" (shape input) (at 203.2 144.78 0) (fields_autoplaced)
-    (effects (font (size 1.27 1.27)) (justify left))
-    (property "Intersheet References" "${INTERSHEET_REFS}" (id 0) (at 214.0798 144.7006 0)
+  (global_label "BTN_Right_UP" (shape input) (at 203.2 144.78 0) (fields_autoplaced)
+    (effects (font (size 1.27 1.27)) (justify left))
+    (property "Intersheet References" "${INTERSHEET_REFS}" (id 0) (at 218.6155 144.7006 0)
       (effects (font (size 1.27 1.27)) (justify left) hide)
     )
@@
     )
   )
-  (global_label "LU" (shape input) (at 201.93 76.2 0) (fields_autoplaced)
+  (global_label "LU" (shape output) (at 201.93 76.2 0) (fields_autoplaced)
     (effects (font (size 1.27 1.27)) (justify left))
     (property "Intersheet References" "${INTERSHEET_REFS}" (id 0) (at 206.7017 76.1206 0)
@@
     )
   )
-  (global_label "Right_DOWN" (shape input) (at 277.495 111.125 180) (fields_autoplaced)
-    (effects (font (size 1.27 1.27)) (justify right))
-    (property "Intersheet References" "${INTERSHEET_REFS}" (id 0) (at 263.8333 111.0456 0)
+  (global_label "BTN_Right_DOWN" (shape input) (at 277.495 111.125 180) (fields_autoplaced)
+    (effects (font (size 1.27 1.27)) (justify right))
+    (property "Intersheet References" "${INTERSHEET_REFS}" (id 0) (at 259.2976 111.0456 0)
       (effects (font (size 1.27 1.27)) (justify right) hide)
     )
@@
     )
   )
-  (global_label "TRAVEL" (shape input) (at 203.2 134.62 0) (fields_autoplaced)
-    (effects (font (size 1.27 1.27)) (justify left))
-    (property "Intersheet References" "${INTERSHEET_REFS}" (id 0) (at 212.205 134.5406 0)
+  (global_label "BTN_TRAVEL" (shape input) (at 203.2 134.62 0) (fields_autoplaced)
+    (effects (font (size 1.27 1.27)) (justify left))
+    (property "Intersheet References" "${INTERSHEET_REFS}" (id 0) (at 216.7407 134.5406 0)
       (effects (font (size 1.27 1.27)) (justify left) hide)
     )
@@
     )
   )
-  (global_label "TRAVEL" (shape input) (at 277.495 102.235 180) (fields_autoplaced)
-    (effects (font (size 1.27 1.27)) (justify right))
-    (property "Intersheet References" "${INTERSHEET_REFS}" (id 0) (at 268.49 102.1556 0)
-      (effects (font (size 1.27 1.27)) (justify right) hide)
-    )
+  (global_label "BTN_TRAVEL" (shape input) (at 277.495 102.235 180) (fields_autoplaced)
+    (effects (font (size 1.27 1.27)) (justify right))
+    (property "Intersheet References" "${INTERSHEET_REFS}" (id 0) (at 263.9543 102.1556 0)
+      (effects (font (size 1.27 1.27)) (justify right) hide)
+    )
